File: ledmerkki2k26.kicad_pcb (KiCad board)
At the start: 2 copper layers, 52.2 x 74.7 mm, 71 parts, among them J1 Conn_01x03_Socket, J2 Conn_01x02_Pin, J3 Conn_01x06_Pin, SW1 SW_Push, U1 ATmega328PB-A, Y1 Resonator

Commit message: move mic out of the way
Parts:
- moved J1 1.48 mm to (112.4, 87.9)
Routing:
- net +5V: track 379.6 -> 381.1 mm
- net /dac: track 70.3 -> 71.0 mm
Other:
- outline, holes or cut-outs redrawn
