File: ledmerkki2k26.kicad_sch (KiCad schematic)
At the start: 66 parts, among them J1 Conn_01x03_Socket, J2 Conn_01x02_Pin, J3 Conn_01x06_Pin, SW1 SW_Push, U1 ATmega328PB-A, Y1 Resonator

Commit message: updates to pcb layout and shape, uart pins exposed
Parts:
- added C14: 500uF, Capacitor_SMD:C_1206_3216Metric_Pad1.33x1.80mm_HandSolder, symbol Device:C
- added J5: uart, Connector_PinSocket_2.54mm:PinSocket_1x03_P2.54mm_Vertical, symbol Connector:Conn_01x03_Socket
- added R3: 500R, LED_SMD:LED_0805_2012Metric_Pad1.15x1.40mm_HandSolder, symbol Device:R
- C1, C10, C11, C12, C13, C2, C3, C4, C5, C6, C7, C8, C9, R1, R2: KiLib_Generator (none) -> SMD_2terminal_chip_molded
- J1: value Conn_01x03_Socket -> mic module header; KiLib_Generator (none) -> connector/pin_header_socket
- J2: value Conn_01x02_Pin -> power header; KiLib_Generator (none) -> connector/pin_header_socket
- J3: value Conn_01x06_Pin -> ISP header; KiLib_Generator (none) -> connector/pin_header_socket
- U1: KiLib_Generator (none) -> package/gullwing
Connections:
- net +5V: now also J3.2 (Pin_2), C14.1; no longer J3.1 (Pin_1)
- net DATA: now also R3.1; no longer D39.3 (DIN)
- net GND: now also J3.1 (Pin_1), C14.2, J5.1 (Pin_1); no longer J3.6 (Pin_6)
- net MISO: now also J3.5 (Pin_5); no longer J3.4 (Pin_4)
- net MOSI: now also J3.6 (Pin_6); no longer J3.5 (Pin_5)
- net SCK: now also J3.4 (Pin_4); no longer J3.3 (Pin_3)
- net UART_RX: now also J5.3 (Pin_3)
- net UART_TX: now also J5.2 (Pin_2)
- net button: now also U1.32 (PD2); no longer U1.10 (PD6)
- net reset: now also J3.3 (Pin_3); no longer J3.2 (Pin_2)
- new net: D39.3 (DIN), R3.2
Other:
- note added: "LED decoupling capacitors"
- moved on the sheet: C10, C11, C12, C13, C3, C4, C5, C6, C7, C8, C9, J1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

Commit message: cap footprint added
Parts:
- C14: footprint Capacitor_SMD:C_1206_3216Metric_Pad1.33x1.80mm_HandSolder -> Capacitor_Tantalum_SMD:CP_EIA-7343-15_Kemet-W_HandSolder
Changed lines of the file:
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@@
 			)
 		)
-		(property "Footprint" "Capacitor_SMD:C_1206_3216Metric_Pad1.33x1.80mm_HandSolder"
+		(property "Footprint" "Capacitor_Tantalum_SMD:CP_EIA-7343-15_Kemet-W_HandSolder"
 			(at -9.1948 -19.05 0)
 			(hide yes)
